Commit message: Tune ToF low obstacle simulation

File: sim_bot/description/palmares_tof_lidar.xacro (robot description, xacro)
@@ -5,5 +5,8 @@
         <parent link="chassis"/>
         <child link="tof_lidar_frame"/>
-        <origin xyz="0.065 0 0.18" rpy="0 0 0"/>
+        <!-- Altura antiga: z=0.18 relativo ao chassis => 0.355 m do chao. -->
+        <!-- Teste anterior: z=-0.025 relativo ao chassis => 0.150 m do chao. -->
+        <!-- Altura atual: z=0.025 relativo ao chassis => 0.200 m do chao. -->
+        <origin xyz="0.065 0 0.025" rpy="0 0 0"/>
     </joint>
     <link name="tof_lidar_frame">

Commit message: Update ToF ramp simulation scenarios
Restore the simulated ToF height to 0.355 m and make setup_sim.bash portable across clone locations.

Widen and extend the 15 degree test ramp with a 60 cm plateau, reposition the following 20 degree ramp, and add the long 15 degree ramp used in the aceleradora world.

File: sim_bot/description/palmares_tof_lidar.xacro (robot description, xacro)
@@ -5,8 +5,7 @@
         <parent link="chassis"/>
         <child link="tof_lidar_frame"/>
-        <!-- Altura antiga: z=0.18 relativo ao chassis => 0.355 m do chao. -->
-        <!-- Teste anterior: z=-0.025 relativo ao chassis => 0.150 m do chao. -->
-        <!-- Altura atual: z=0.025 relativo ao chassis => 0.200 m do chao. -->
-        <origin xyz="0.065 0 0.025" rpy="0 0 0"/>
+        <!-- Altura atual: z=0.18 relativo ao chassis => 0.355 m do chao. -->
+        <!-- Alturas testadas: z=-0.025 => 0.150 m; z=0.025 => 0.200 m do chao. -->
+        <origin xyz="0.065 0 0.18" rpy="0 0 0"/>
     </joint>
     <link name="tof_lidar_frame">
